File: vmuzero_SEPS525_V1_0_ICHG100.sch (EAGLE design)
At the start: 63 parts, among them CN1 PIEZO, J1 USB_MICRO_B, U1 BQ24075QRGTRQ1, U2 TLV61046ADBV, U3 DD-160128FC-2B, U4 LT3469TS8, U5 RPI-ZERO_GPIO

Commit message: Add files via upload
Parts:
- R10: value NOSTUFF -> 10k
- R11: value 10k -> NOSTUFF
- R2: value 590 -> 5.9k
Other:
- note added: "EN1 EN2 Current 0 0 100mA 1 0 500mA 0 1 ILIM 1 1 Standby"
- note removed: "EN1 EN2 Current 0 0 100mA 1 0 500mA 0 1 ISET 1 1 Standby"
Changed lines of the file:
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@@
 <setting verticaltext="up"/>
 </settings>
-<grid distance="0.1" unitdist="inch" unit="inch" style="lines" multiple="1" display="yes" altdistance="0.01" altunitdist="inch" altunit="inch"/>
+<grid distance="0.1" unitdist="inch" unit="inch" style="lines" multiple="1" display="no" altdistance="0.01" altunitdist="inch" altunit="inch"/>
 <layers>
 <layer number="1" name="Top" color="4" fill="1" visible="no" active="no"/>
@@
 <part name="R1" library="microbuilder" deviceset="RESISTOR" device="_0805MP" value="1.1k"/>
 <part name="SUPPLY7" library="supply2" deviceset="GND" device=""/>
-<part name="R2" library="microbuilder" deviceset="RESISTOR" device="_0805MP" value="590"/>
+<part name="R2" library="microbuilder" deviceset="RESISTOR" device="_0805MP" value="5.9k"/>
 <part name="SUPPLY8" library="supply2" deviceset="GND" device=""/>
 <part name="R3" library="microbuilder" deviceset="RESISTOR" device="_0805MP" value="NOSTUFF"/>
@@
 <part name="R8" library="microbuilder" deviceset="RESISTOR" device="_0805MP" value="NOSTUFF"/>
 <part name="R9" library="microbuilder" deviceset="RESISTOR" device="_0805MP" value="10k"/>
-<part name="R10" library="microbuilder" deviceset="RESISTOR" device="_0805MP" value="NOSTUFF"/>
-<part name="R11" library="microbuilder" deviceset="RESISTOR" device="_0805MP" value="10k"/>
+<part name="R10" library="microbuilder" deviceset="RESISTOR" device="_0805MP" value="10k"/>
+<part name="R11" library="microbuilder" deviceset="RESISTOR" device="_0805MP" value="NOSTUFF"/>
 <part name="SUPPLY12" library="supply2" deviceset="GND" device=""/>
 <part name="SUPPLY13" library="supply2" deviceset="GND" device=""/>
@@
  0   0   100mA
  1   0   500mA
- 0   1   ISET
+ 0   1   ILIM
  1   1   Standby</text>
 <text x="30.48" y="63.5" size="1.778" layer="97">S1
