File: vmuzero_SEPS525_V1_8_1.sch (EAGLE design)
At the start: 63 parts, among them CN1 PIEZO, J1 USB_MICRO_B, U1 BQ24075QRGTRQ1, U2 TLV61046ADBV, U3 DD-160128FC-2B, U4 LT3469TS8, U5 RPI-ZERO_GPIO

Commit message: V2 prototype
Parts:
- removed CHG: YELLOW, microbuilder:LED0805_NOOUTLINE
- removed L2: 47uH, vmuzero:INDUCTOR_LQH32C
- removed PGOOD: BLUE, microbuilder:LED0805_NOOUTLINE
- removed R11: NOSTUFF, microbuilder:RESISTOR_0805MP
- removed R12: 100k, microbuilder:RESISTOR_0805MP
- removed R19: 16k, microbuilder:RESISTOR_0805MP
- removed U4: LT3469TS8, vmuzero:LT3469TS8
- added C11: 0.1uF, microbuilder:CAP_CERAMIC_0805MP
- added C12: 10uF, microbuilder:CAP_CERAMIC_0805MP
- added C22: 0.1uF/10V, microbuilder:CAP_CERAMIC_0805MP
- added DZ1, DZ2: SP1003-01, vmuzero:SP1003-01D
- added DZ3: SP1001-04J, vmuzero:SP1001-04J
- added Q1: SSM3J15FU, vmuzero:MOSFET_PCH-SSM3J15FU
- added Q2: SSM3K7002CFU, vmuzero:MOSFET_NCH-SSM3K7002CFU
- added R27, R31: 47k, microbuilder:RESISTOR_0805MP
- added R28: 100, microbuilder:RESISTOR_0805MP
- added R29: 20k, microbuilder:RESISTOR_0805MP
- added TP1: TPTP14SQ, testpad:TPTP14SQ
- added TP11, TP12, TP13, TP14, TP15, TP16, TP18, TP19, TP2, TP20, TP22, TP23, TP24, TP29, TP30, TP32, TP34, TP36, TP37, TP39, TP4, TP6, TP7, TP9: TPTP14R, testpad:TPTP14R
- added U6: MIC94064YC6, vmuzero:MIC94064YC6
- added U7: LM358ADR, vmuzero:LM358ADR
- C20: value 1uF -> 1uF/16V
- C21: value 0.47uF/35V -> 1uF
- C23: value 5.6nF -> 1u
- D1: value SP1003-01 -> YELLOW; device vmuzero:SP1003-01D -> microbuilder:LED0805_NOOUTLINE
- D2: value SP1003-01 -> GREEN; device vmuzero:SP1003-01D -> microbuilder:LED0805_NOOUTLINE
- D3: value SP1001-04J -> BLUE; device vmuzero:SP1001-04J -> microbuilder:LED0805_NOOUTLINE
- J1: device vmuzero:USB_MICRO-B_CUI_MIBH2 -> vmuzero:USB_MICRO-B_AMP_10118192
- L1: device vmuzero:INDUCTOR_LQH2 -> vmuzero:INDUCTOR_CIG22L
- R1: value 1.1k -> 2k
- R13: value 1.2M -> 1.21M
- R2: value 5.9k -> 10k
- R20: value 270k -> 47k
- R21: value 16k -> 47k
- R22: value 20k -> 100k
- R23: value 110k -> 47k
- R24: value 0 -> 100
- R3: value NOSTUFF -> 100k
- R4: value 10k -> 560k
- R6: value 1.5k -> 1.8k
- R7: value 100k -> 1.5k
- R8: value NOSTUFF -> 0
- R9: value 10k -> 1k
- U1: value BQ24075QRGTRQ1 -> MCP73833-UN; device SparkFun-IC-Power:BQ24075 -> vmuzero:MCP73833-UN
- U5: value RPI-ZERO_GPIO -> RPI-ZERO_OUTLINE; device vmuzero:RPI-ZERO_GPIO -> vmuzero:RPI-ZERO_OUTLINE
- renumbered D4 to DZ4
Connections:
- removed net N$14: L2.2, U4.SW
- removed net N$17: C23.P$1, R23.1, R24.1, U4.OUT
- removed net N$18: R22.2, R23.2, U4.IN-
- removed net N$19: CN1.1, R24.2
- removed net N$4: R12.1, S1.O
- removed net PM_CE: R7.2, U1.!CE!
- removed net PM_EN1: R8.1, R9.2, U1.EN1
- removed net PM_EN2: R10.1, R11.2, U1.EN2
- removed net PM_ILIM: R1.2, U1.ILIM
- removed net PM_ISET: R2.2, U1.ISET
- removed net PM_SYSOFF: D2.C, S1.P, U1.SYSOFF
- removed net PM_TMR: R3.2, U1.TMR
- removed net PM_TS: R4.2, U1.TS
- removed net VCC_AMP: C21.P$2, R20.2, U4.VCC
- new net N$12: R29.2, R31.1, U7A.-IN
- new net N$13: C21.P$2, R29.1
- new net N$22: Q1.D, R10.1, R4.2
- new net N$3: C23.P$2, R25.1
- new net PM_NTC: R2.2, U1.THERM
- new net PM_PROG: R1.2, U1.PROG
- new net PM_SHUTDOWN: R9.2, TP29.TP
- new net PM_STAT1: D1.C, U1.STAT1
- new net PM_STAT2: D2.C, U1.STAT2
- new net PM_SYSON: C12.P$1, R10.2, U6.EN
- new net PM_SYSON_L: C11.P$1, DZ2.C, Q1.G, R3.1, R8.1, S1.P
- new net VOUTN: R23.2, R28.1, U7B.OUT
- new net VOUTN_R: CN1.1, R28.2
- new net VOUTP: R24.1, R27.2, R31.2, U7A.OUT
- new net VOUTP_R: CN1.2, R24.2
- new net V_AMP_CM: C22.P$2, R20.1, R21.2, R22.2, U7B.+IN
- net 14V: now also R26.1
- net 3.3V: now also TP1.TP; no longer U5.3V3
- net GND: now also C11.P$2, C12.P$2, C22.P$1, D3.C, DZ1.A, DZ2.A, DZ3.A, Q2.S, R21.1, TP14.TP, TP20.TP, TP30.TP, TP34.TP, TP39.TP, TP6.TP, TP9.TP, U6.GND, U7P.V-; no longer C23.P$2, CN1.2, D1.A, D2.A, D3.A, R11.1, R19.2, R22.1, R3.1, R7.1, R9.1, U1.EP, U4.GND, U5.GND@1, U5.GND@2, U5.GND@3, U5.GND@4, U5.GND@5, U5.GND@6, U5.GND@7, U5.GND@8
- net KEY_A: now also TP7.TP; no longer U5.GPIO4
- net KEY_B: now also TP32.TP; no longer U5.GPIO12
- net KEY_DOWN: now also DZ3.C4, TP13.TP; no longer D3.C2, U5.GPIO27
- net KEY_LEFT: now also DZ3.C1, TP11.TP; no longer D3.C1, U5.GPIO17
- net KEY_RIGHT: now also DZ3.C2, TP15.TP; no longer D3.C4, U5.GPIO22
- net KEY_SELECT: now also TP36.TP; no longer U5.GPIO16
- net KEY_START: now also TP37.TP; no longer U5.GPIO26
- net KEY_UP: now also DZ3.C3, TP16.TP; no longer D3.C3, U5.GPIO23
- net N$1: now also D1.A, R5.1; no longer CHG.C, U1.!CHG!
- net N$16: now also R23.1, R27.1, U7B.-IN; no longer R19.1, R20.1, U4.FB
- net N$2: now also Q2.D, R9.1; no longer PGOOD.C, U1.!PGOOD!
- net N$20: now also R22.1, U7A.+IN; no longer R21.1
- net N$21: now also Q2.G, R8.2; no longer R21.2, U4.IN+
- net N$5: now also D3.A, R7.1; no longer PGOOD.A, R6.1
- net N$6: now also D2.A, R6.1; no longer CHG.A, R5.1
- net OLED_CS: now also TP24.TP; no longer U5.!CE0!/GPIO8
- net OLED_DC: now also TP22.TP; no longer U5.GPIO25
- net OLED_MOSI: now also TP19.TP; no longer U5.GPIO10/MOSI
- net OLED_RES: now also TP18.TP; no longer U5.GPIO24
- net OLED_SCLK: now also TP23.TP; no longer U5.GPIO11/SCLK
- net PWM0: now also C23.P$1, TP12.TP; no longer R25.1, U5.GPIO18
- net VSYS: now also R7.2, U6.VOUT; no longer R10.2, R26.1, R5.2, R6.2, R8.2, U1.OUT
- net VSYS_AMP: now also R20.2, U7P.V+; no longer L2.1, U4.VIN
- net VSYS_RPI: now also TP2.TP, TP4.TP; no longer U5.5V0@1, U5.5V0@2
- net V_BATT: now also Q1.S, R3.2, R5.2, R6.2, U1.VBAT, U6.VIN; no longer R12.2, U1.BAT
- net V_USB: now also DZ1.C, U1.VDD; no longer D1.C, U1.IN
Other:
- note added: "BW1 Fc1 = 8Hz"
- note added: "BW2 Fc2 = 16Hz"
- note added: "BW3 Fc3 = 17kHz"
- note added: "CHARGE"
- note added: "CHG_DONE"
- note added: "Gain = 10.5dB"
- note added: "MAX 2mA @ 14.5V"
- note added: "PROG Charge Current = 1000V/R_PROG 2.0kΩ 500mA 2.9kΩ 350mA 6.8kΩ 150mA"
- note added: "VOUT = 0.795V x (1 + R13/R14) VOUT = 14.25V"
- note added: "VSYS"
- note removed: "EN1 EN2 Current 0 0 100mA 1 0 500mA 0 1 ILIM 1 1 Standby"
- note removed: "Low Pass Filter Fc = 1/(2Pi x RC) = 17kHz"
- note removed: "MAX 31mA @ 3.7V"
- note removed: "S1 0 ON 1 OFF"
- note removed: "ToDo: Add DC block capacitor"
- note removed: "VCC = 1.23 x (1 + R2/R1) = 21.99V"
- note removed: "VOUT = 0.795V x (1 + R13/R14) VOUT = 14.14V"
- moved on the sheet: C1, C2, C20, C21, C23, C3, CN1, R1, R10, R2, R20, R21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
